File: HW/phloggerV2/phloggerV2.sch (KiCad schematic (older format))
At the start: 30 parts, among them J1 BATTERI CON, J2 boost_conv_ena, J3 PH_PROBE, J4 GPS, U1 74HCT541, U2 pro-mini-deek, U3 LM321, U4 DS3231, U5 3-pin-BoostConv

Commit message: kicad 5
Parts:
- BT1: symbol Battery_Cell -> device:Battery_Cell
- C1, C2, C3, C4, C5, C6: symbol C_Small -> device:C_Small
- C7: symbol CP -> device:CP
- D1: symbol SD-BREAKOUT -> Peters:SD-BREAKOUT
- J1: symbol Screw_Terminal_1x02 -> phloggerV2-rescue:Screw_Terminal_1x02
- J2: symbol CONN_01X01 -> phloggerV2-rescue:CONN_01X01
- J3: symbol Screw_Terminal_1x04 -> phloggerV2-rescue:Screw_Terminal_1x04
- J4: symbol CONN_01X04 -> phloggerV2-rescue:CONN_01X04
- R1, R2, R3, R4: symbol R -> device:R
- TP1, TP2, TP3, TP4, TP5, TP6, TP7, TP8: symbol TEST -> phloggerV2-rescue:TEST
- U1: symbol 74HCT541 -> Peters:74HCT541
- U2: symbol pro-mini-deek -> Peters:pro-mini-deek
- U3: symbol LM321 -> linear:LM321
- U4: symbol DS3231 -> phloggerV2-rescue:DS3231
- U5: symbol 3-pin-BoostConv -> Peters:3-pin-BoostConv
