File: HW/Version3/GPSBoard/gpsBoard/gpsBoard.sch (KiCad schematic (older format))
At the start: 12 parts

Commit message: board
Parts:
- removed C? (x2): 22pf, Capacitors_SMD:C_0805_HandSoldering, symbol C
- removed JP?: Jumper, Pin_Headers:Pin_Header_Straight_1x03_Pitch2.54mm, symbol Jumper
- removed U?: ATMEGA328P-AU-Arduino, Housings_QFP:TQFP-32_7x7mm_Pitch0.8mm, symbol ATMEGA328P-AU-Arduino
- removed Y?: 8MHZ, Crystals:Crystal_HC18-U_Vertical, symbol Crystal
- added C2: CP, symbol device:CP
- added J1, J2: Screw_Terminal_01x03, TerminalBlock_Phoenix:TerminalBlock_Phoenix_PT-3.5mm_3pol, symbol Connector:Screw_Terminal_01x03
- added Q1: Si4435, Housings_SOIC:SOIC-8_3.9x4.9mm_Pitch1.27mm, symbol Peters:Si4435
- added R2: 100K, symbol device:R
- added SW1: SW_Push, symbol Switch:SW_Push
- added U2: GY-NEO6MV2, Libs:GY-NEO6MV2 GPS Module, symbol Peters:GY-NEO6MV2
- added U?: ATTINY85-20PU, Housings_DIP:DIP-8_W7.62mm, symbol atmel:ATTINY85-20PU
- 1U1: renamed from 1U?; symbol C -> device:C
- C1, C4: renamed from C?; symbol C -> device:C
- C3: renamed from C?; symbol CP -> device:CP
- FTDI1: renamed from FTDI?; symbol CONN_01X06 -> gpsBoard-rescue:CONN_01X06-pro-mini-rescue
- ISP1: renamed from ISP?; symbol ISP-header -> gpsBoard-rescue:ISP-header-pro-mini-rescue
- R1: renamed from R?; symbol R -> device:R
Connections:
- net labels added: +3V3, powerOn
- wire segments 30 -> 43
