File: HW/Version3/Main/Main.sch (KiCad schematic (older format))
At the start: 61 parts, among them J1 V_Batt_in, J2 SD_Card_Main, J3 SD_Card_Backup, J4 Vbat, J5 Thermistor_10K, J6 ExternalSwiches, Q1 Si4435, U1 XC6206P332MR, U10 EZO_BNC, U2 XC6206P332MR, U3 GY-NEO6MV2, U4 ADS1115-temp, U5 DS18S20_, U6 Bluepill, U7 AT24CS32-SSHM, U8 OLED_128x32_i2c, U9 EZ_PH

Commit message: Board
Parts:
- removed Q1: Si4435, Housings_SOIC:SOIC-8_3.9x4.9mm_Pitch1.27mm, symbol Peters:Si4435
- added Q?: IRF7341, Housings_SOIC:SOIC-8_3.9x4.9mm_Pitch1.27mm, symbol Peters:IRF7341
Changed lines of the file:
@@
-$EndComp
-$Comp
-L Peters:Si4435 Q1
-U 1 1 5B2F64C6
-P 3350 7150
-F 0 "Q1" H 3556 7196 50  0000 L CNN
-F 1 "Si4435" H 3556 7105 50  0000 L CNN
-F 2 "Housings_SOIC:SOIC-8_3.9x4.9mm_Pitch1.27mm" H 3100 7450 50  0001 C CNN
-F 3 "https://www.vishay.com/docs/72123/72123.pdf" H 3200 7550 50  0001 C CNN
-	1    3350 7150
-	-1   0    0    -1
 $EndComp
 $Comp
@@
 	3250 6350 3250 6450
 Connection ~ 2550 6350
-Wire Wire Line
-	3250 7450 3250 7350
 $Comp
 L device:R R3
@@
 	1    0    0    -1
 $EndComp
-Wire Wire Line
-	3550 7150 3650 7150
 Wire Wire Line
 	3650 7150 3650 7200
@@
 Wire Wire Line
 	5900 7250 6650 7250
+$Comp
+L Peters:IRF7341 Q?
+U 1 1 5B4CBA24
+P 3350 7150
+F 0 "Q?" H 3540 7203 60  0000 L CNN
+F 1 "IRF7341" H 2900 7250 60  0000 L CNN
+F 2 "Housings_SOIC:SOIC-8_3.9x4.9mm_Pitch1.27mm" H 3400 7800 60  0001 C CNN
+F 3 "https://www.infineon.com/dgdl/irf7341.pdf?fileId=5546d462533600a4015355f636411b5d" H 3150 8100 60  0001 C CNN
+	1    3350 7150
+	-1   0    0    -1
+$EndComp
+Wire Wire Line
+	3250 7350 3250 7450
+Wire Wire Line
+	3450 7150 3650 7150
 $EndSCHEMATC

Commit message: Layout beginning
Parts:
- removed J2: SD_Card_Main, symbol Connector:SD_Card
- removed J3: SD_Card_Backup, symbol Connector:SD_Card
- removed J5: Thermistor_10K, TerminalBlock_Phoenix:TerminalBlock_Phoenix_PT-3.5mm_3pol, symbol Connector:Screw_Terminal_01x03
- removed J6: ExternalSwiches, TerminalBlock_Phoenix:TerminalBlock_Phoenix_PT-3.5mm_4pol, symbol Connector:Screw_Terminal_01x04
- removed R5, R6, R7, R8: 20K, Resistors_SMD:R_0805_HandSoldering, symbol device:R_Small
- removed U4: ADS1115-temp, Libs:ADS1115-Breakout, symbol Peters:ADS1115
- removed U5: DS18S20_, digikey-footprints:TO-92-3, symbol dk_Temperature-Sensors-Analog-and-Digital-Output:DS18S20_
- added C28: 100n, Capacitor_SMD:C_0805_2012Metric_Pad1.15x1.40mm_HandSolder, symbol device:C_Small
- added J3, J5: Spare, Connector_PinHeader_2.54mm:PinHeader_1x04_P2.54mm_Vertical, symbol Connector:Conn_01x04_Female
- added J4: Ext temp, TerminalBlock_Phoenix:TerminalBlock_Phoenix_PT-1,5-3-3.5-H_1x03_P3.50mm_Horizontal, symbol Connector:Screw_Terminal_01x03
- added J6: ExtSw, TerminalBlock_TE-Connectivity:TerminalBlock_TE_282834-5_1x05_P2.54mm_Horizontal, symbol Connector:Screw_Terminal_01x05
- added M1: BOX_Biltema_70x70_IP67, Libs:Box_Biltema_70x70mm_IP67, symbol Peters:BOX_Biltema_70x70_IP67
- added U12: SN74LVC2G14, Package_TO_SOT_SMD:SOT-23-6_Handsoldering, symbol Peters:SN74LVC2G14
- added U13: MAX17043Breakout, Libs:MAX17043-Breakout, symbol Peters:MAX17043Breakout
- added U2, U3: SdmicroBreakout, Libs:MicroSD_Card_Breakout_Horizontal, symbol Peters:SdmicroBreakout
- added U6: ADM1023, Package_SO:TSSOP-16_4.4x5mm_P0.65mm, symbol Peters:ADM1023
- C1: renamed from C3; footprint Capacitors_SMD:CP_Elec_4x5.3 -> Capacitor_SMD:CP_Elec_4x5.3
- C10: renamed from C12; footprint Capacitors_SMD:C_0805_HandSoldering -> Capacitor_SMD:C_0805_2012Metric_Pad1.15x1.40mm_HandSolder
- C11: renamed from C8; footprint Capacitors_SMD:C_0805_HandSoldering -> Capacitor_SMD:C_0805_2012Metric_Pad1.15x1.40mm_HandSolder
- C12: renamed from C6; footprint Capacitors_SMD:C_0805_HandSoldering -> Capacitor_SMD:C_0805_2012Metric_Pad1.15x1.40mm_HandSolder
- C13, C14, C15, C17, C19, C20, C21, C22, C23, C25, C26: footprint Capacitors_SMD:C_0805_HandSoldering -> Capacitor_SMD:C_0805_2012Metric_Pad1.15x1.40mm_HandSolder
- C16, C2, C24, C27: footprint Capacitors_SMD:CP_Elec_4x5.3 -> Capacitor_SMD:CP_Elec_4x5.3
- C18: value 100n -> 680p; footprint Capacitors_SMD:C_0805_HandSoldering -> Capacitor_SMD:C_0805_2012Metric_Pad1.15x1.40mm_HandSolder
- C3: renamed from C1; footprint Capacitors_SMD:C_0805_HandSoldering -> Capacitor_SMD:C_0805_2012Metric_Pad1.15x1.40mm_HandSolder
- C4: renamed from C7; footprint Capacitors_SMD:C_0805_HandSoldering -> Capacitor_SMD:C_0805_2012Metric_Pad1.15x1.40mm_HandSolder
- C5: renamed from C9; footprint Capacitors_SMD:CP_Elec_4x5.3 -> Capacitor_SMD:CP_Elec_4x5.3
- C6: renamed from C5; footprint Capacitors_SMD:C_0805_HandSoldering -> Capacitor_SMD:C_0805_2012Metric_Pad1.15x1.40mm_HandSolder
- C7: renamed from C10; footprint Capacitors_SMD:C_0805_HandSoldering -> Capacitor_SMD:C_0805_2012Metric_Pad1.15x1.40mm_HandSolder
- C8: renamed from C11; footprint Capacitors_SMD:C_0805_HandSoldering -> Capacitor_SMD:C_0805_2012Metric_Pad1.15x1.40mm_HandSolder
- C9: renamed from C4; footprint Capacitors_SMD:C_0805_HandSoldering -> Capacitor_SMD:C_0805_2012Metric_Pad1.15x1.40mm_HandSolder
- F1: footprint Fuse_Holders_and_Fuses:Fuse_SMD1206_HandSoldering -> Libs:LittleFuse_110F_24V
- J1: footprint TerminalBlock_Phoenix:TerminalBlock_Phoenix_PT-3.5mm_3pol -> TerminalBlock_Phoenix:TerminalBlock_Phoenix_PT-1,5-3-3.5-H_1x03_P3.50mm_Horizontal
- J2: renamed from J4; footprint TerminalBlock_Phoenix:TerminalBlock_Phoenix_PT-3.5mm_3pol -> Connector_PinHeader_2.54mm:PinHeader_1x01_P2.54mm_Vertical
- Q1: renamed from Q?; footprint Housings_SOIC:SOIC-8_3.9x4.9mm_Pitch1.27mm -> Package_SO:SOIC-8_3.9x4.9mm_P1.27mm
- R1: renamed from R2; footprint Resistors_SMD:R_1210_HandSoldering -> Resistor_SMD:R_1210_3225Metric_Pad1.42x2.65mm_HandSolder
- R10: renamed from R12; footprint Resistors_SMD:R_0805_HandSoldering -> Resistor_SMD:R_0805_2012Metric_Pad1.15x1.40mm_HandSolder
- R2: renamed from R1; footprint Resistors_SMD:R_1210_HandSoldering -> Resistor_SMD:R_1210_3225Metric_Pad1.42x2.65mm_HandSolder
- R3: footprint Resistors_SMD:R_0805_HandSoldering -> Resistor_SMD:R_0805_2012Metric_Pad1.15x1.40mm_HandSolder
- R4: value 4k7 -> 82K; footprint Resistors_SMD:R_0805_HandSoldering -> Resistor_SMD:R_0805_2012Metric_Pad1.15x1.40mm_HandSolder
- R7: renamed from R9; footprint Resistors_SMD:R_0805_HandSoldering -> Resistor_SMD:R_0805_2012Metric_Pad1.15x1.40mm_HandSolder
- R8: renamed from R10; footprint Resistors_SMD:R_0805_HandSoldering -> Resistor_SMD:R_0805_2012Metric_Pad1.15x1.40mm_HandSolder
- R9: renamed from R11; footprint Resistors_SMD:R_0805_HandSoldering -> Resistor_SMD:R_0805_2012Metric_Pad1.15x1.40mm_HandSolder
- TP1: renamed from TP2; footprint Connectors_TestPoints:Test_Point_Pad_d2.0mm -> TestPoint:TestPoint_Loop_D1.80mm_Drill1.0mm_Beaded
- TP2: renamed from TP1; footprint Connectors_TestPoints:Test_Point_Pad_d2.0mm -> TestPoint:TestPoint_Loop_D1.80mm_Drill1.0mm_Beaded
- TP3: renamed from TP4; footprint Connectors_TestPoints:Test_Point_Pad_d2.0mm -> TestPoint:TestPoint_Loop_D1.80mm_Drill1.0mm_Beaded
- TP4: renamed from TP3; footprint Connectors_TestPoints:Test_Point_Pad_d2.0mm -> TestPoint:TestPoint_Loop_D1.80mm_Drill1.0mm_Beaded
- U1: footprint TO_SOT_Packages_SMD:SOT-23_Handsoldering -> Package_TO_SOT_SMD:SOT-23_Handsoldering
- U4: renamed from U2; footprint TO_SOT_Packages_SMD:SOT-23_Handsoldering -> Package_TO_SOT_SMD:SOT-23_Handsoldering
- U8: renamed from U7; footprint Housings_SOIC:SOIC-8_3.9x4.9mm_Pitch1.27mm -> Package_SO:SOIC-8_3.9x4.9mm_P1.27mm
- U9: renamed from U8; footprint Pin_Headers:Pin_Header_Straight_1x04_Pitch2.54mm -> Connector_PinHeader_2.54mm:PinHeader_1x04_P2.54mm_Vertical
- renumbered U9 to U10, U10 to U11, U3 to U5, U6 to U7
Connections:
- net labels added: ADMStby
- net labels removed: InternalTemp
- wire segments 149 -> 143
- no-connect marks 2 -> 13
Other:
- note added: "addr:0x18"
