File: HW/Version4/Board/Board.sch (KiCad schematic (older format))
At the start: 62 parts, among them J1 V_Batt_in, J2 Vbat, J3 Spare, J4 Ext temp, J5 Spare, J6 ExtSw, M1 BOX_Biltema_70x70_IP67, Q1 IRF7341, U1 XC6206P332MR, U10 EZ_PH, U11 EZO_BNC, U12 SN74LVC2G14, U13 MAX17043Breakout, U2 SdmicroBreakout, U3 SdmicroBreakout, U4 XC6206P332MR, U5 GY-NEO6MV2, U6 ADM1023, U7 Bluepill, U8 AT24CS32-SSHM, U9 OLED_128x32_i2c

Commit message: V4 started
Parts:
- renumbered C27 to C?, C26 to C?, C25 to C?, C24 to C?, C8 to C?, C5 to C?, C17 to C?, C16 to C?, C19 to C?, C14 to C?, C22 to C?, C13 to C?, C10 to C?, C9 to C?, C2 to C?, C6 to C?, C1 to C?, C11 to C?, C12 to C?, C4 to C?, C3 to C?, C7 to C?, C21 to C?, C20 to C?, C15 to C?, C18 to C?, C23 to C?, C28 to C?, F1 to F?, J1 to J?, J2 to J?, J4 to J?, J5 to J?, J3 to J?, J6 to J?, M1 to M?, Q1 to Q?, R7 to R?, R8 to R?, R3 to R?, R2 to R?, R1 to R?, R9 to R?, R10 to R?, R4 to R?, TP3 to TP?, TP1 to TP?, TP2 to TP?, TP4 to TP?, U7 to U?, U11 to U?, U5 to U?, U9 to U?, U10 to U?, U4 to U?, U1 to U?, U8 to U?, U6 to U?, U13 to U?, U2 to U?, U3 to U?, U12 to U?
Other:
- note added: "SPI oled\nvertical SD cards\nBetter GPS mgnt\nBetter cabling\nMore temp sense\nPull out SPI + I2c port for future\nmcu voltage watchdog\n"

Commit message: V4 beginning
Parts:
- removed C? (x4): 10u, Capacitor_SMD:CP_Elec_4x5.3, symbol Main-rescue:CP1_Small-device
- removed C? (x9): 100n, Capacitor_SMD:C_0805_2012Metric_Pad1.15x1.40mm_HandSolder, symbol Main-rescue:C_Small-device
- removed C? (x4): 1u, Capacitor_SMD:C_0805_2012Metric_Pad1.15x1.40mm_HandSolder, symbol Main-rescue:C_Small-device
- removed C?: 680p, Capacitor_SMD:C_0805_2012Metric_Pad1.15x1.40mm_HandSolder, symbol Main-rescue:C_Small-device
- removed F?: Polyfuse, Libs:LittleFuse_110F_24V, symbol Main-rescue:Polyfuse-device
- removed J?: V_Batt_in, TerminalBlock_Phoenix:TerminalBlock_Phoenix_PT-1,5-3-3.5-H_1x03_P3.50mm_Horizontal, symbol Connector:Screw_Terminal_01x03
- removed J?: Vbat, Connector_PinHeader_2.54mm:PinHeader_1x01_P2.54mm_Vertical, symbol Connector:Conn_01x01_Female
- removed J?: Ext temp, TerminalBlock_Phoenix:TerminalBlock_Phoenix_PT-1,5-3-3.5-H_1x03_P3.50mm_Horizontal, symbol Connector:Screw_Terminal_01x03
- removed J? (x2): Spare, Connector_PinHeader_2.54mm:PinHeader_1x04_P2.54mm_Vertical, symbol Connector:Conn_01x04_Female
- removed Q?: IRF7341, Package_SO:SOIC-8_3.9x4.9mm_P1.27mm, symbol Peters:IRF7341
- removed R?: 4K7, Resistor_SMD:R_0805_2012Metric_Pad1.15x1.40mm_HandSolder, symbol Main-rescue:R-device
- removed R? (x2): 0R1, Resistor_SMD:R_1210_3225Metric_Pad1.42x2.65mm_HandSolder, symbol Main-rescue:R-device
- removed R?: 82K, Resistor_SMD:R_0805_2012Metric_Pad1.15x1.40mm_HandSolder, symbol Main-rescue:R-device
- removed TP? (x4): Test_Point, TestPoint:TestPoint_Loop_D1.80mm_Drill1.0mm_Beaded, symbol Main-rescue:Test_Point-Connector
- removed U?: EZO_BNC, Libs:EZO_BNC, symbol Peters:EZO_BNC
- removed U?: GY-NEO6MV2, Libs:GY-NEO6MV2 GPS Module, symbol Peters:GY-NEO6MV2
- removed U?: OLED_128x32_i2c, Connector_PinHeader_2.54mm:PinHeader_1x04_P2.54mm_Vertical, symbol Peters:OLED_128x32_i2c
- removed U?: EZ_PH, Libs:atlas-scientific.ezo.ph, symbol Peters:EZ_PH
- removed U? (x2): XC6206P332MR, Package_TO_SOT_SMD:SOT-23_Handsoldering, symbol Peters:XC6206P332MR
- removed U?: ADM1023, Package_SO:TSSOP-16_4.4x5mm_P0.65mm, symbol Peters:ADM1023
- removed U?: MAX17043Breakout, Libs:MAX17043-Breakout, symbol Peters:MAX17043Breakout
- removed U? (x2): SdmicroBreakout, Libs:MicroSD_Card_Breakout_Horizontal, symbol Peters:SdmicroBreakout
- added C1, C3: 10u, Capacitor_SMD:CP_Elec_4x5.3, symbol Board-rescue:CP1_Small-device-Main-rescue
- added C15, C2, C4: 100n, Capacitor_SMD:C_0805_2012Metric_Pad1.15x1.40mm_HandSolder, symbol Board-rescue:C_Small-device-Main-rescue
- added J1: SPI2Breakout, Connector_PinHeader_2.54mm:PinHeader_1x06_P2.54mm_Vertical, symbol Connector:Conn_01x06_Male
- added J2: I2cBreakout, Connector_PinHeader_2.54mm:PinHeader_1x04_P2.54mm_Vertical, symbol Connector:Conn_01x04_Male
- added U1: NRF2401+, Libs:NRFl0breakout, symbol Peters:NRF2401+
- added U11: OLED_128x64_SPI_0.96\", Libs:OLED_128x64_i2c, symbol Peters:OLED_128x64_SPI_0.96"
- added U6: LM321, Package_TO_SOT_SMD:SOT-23-5, symbol Amplifier_Operational:LM321
- C11, C13, C14, C16, C17, C18, C19, C21: renamed from C?; symbol Main-rescue:C_Small-device -> Board-rescue:C_Small-device-Main-rescue
- C12, C20: renamed from C?; symbol Main-rescue:CP1_Small-device -> Board-rescue:CP1_Small-device-Main-rescue
- R10, R7, R8, R9: renamed from R?; symbol Main-rescue:R-device -> Board-rescue:R-device-Main-rescue
- U8: renamed from U?; symbol Main-rescue:AT24CS32-SSHM-memory -> Board-rescue:AT24CS32-SSHM-memory-Main-rescue
- gave numbers to parts that had none: 4
Connections:
- net GND: now also C1.2, C15.2, C2.2, C3.2, C4.2, J1.1 (Pin_1), J2.1 (Pin_1), U1.1 (GND), U11.1 (GND), U6.2 (V-)
- net MISO1: now also U1.7 (MI)
- net MISO2: now also J1.3 (Pin_3)
- net MOSI1: now also U1.6 (MO)
- net MOSI2: now also J1.2 (Pin_2)
- net SCK1: now also U1.5 (SCK)
- net SCK2: now also J1.4 (Pin_4)
- net SCL: now also J2.2 (Pin_2)
- net SDA: now also J2.3 (Pin_3)
- net VCC: now also C1.1, C15.1, C2.1, C3.1, C4.1, J1.6 (Pin_6), J2.4 (Pin_4), U1.2 (Vcc), U11.2 (VCC), U6.5 (V+)
- net OLED_SS: now reaches U7.13 (PB0_ADC8_PWM)
- net GPS-RX: now reaches U7.15 (PB10_SCL2_TX3_5V)
- net SpareSS: now reaches U7.25 (PA8_PWM_5V)
- net SpareSS: now also J1.5 (Pin_5)
- net BtnDN: now reaches U7.27 (PA10_RX1_PWM_5V)
- net BtnDN: now also U10.4 (Y)
- net CE-NRF: now reaches U7.30 (PA15_5V)
- net CE-NRF: now also U1.3 (CE)
- net CSN-NRF: now reaches U7.31 (PB3_5V)
- net CSN-NRF: now also U1.4 (CSN)
- net IRQNRF: now reaches U7.32 (PB4_5V)
- net 1WireDHT: now reaches U7.33 (PB5)
- net 1WireDHT: now also U7.8 (PA3_ADC3_PWM_RX2)
- net at U7.5 (PA0_ADC0_PMW): now also U6.3 (-), U6.4
- net Battery and power/Battcharging: now reaches U7.6 (PA1_ADC1_PWM)
- net MAX6475L_IO: now reaches U7.7 (PA2_ADC2_PWM_TX2)
- net MAX6475L_IO: now also U7.36 (PB8_PWM_5V)
- removed net Btn: U10.4 (Y), U7.36 (PB8_PWM_5V)
- net LogginTypeSw renamed BtnUP
- new net Battery and power/BatteryTempAlert¨: U6.1 (+)
- new net IRQ-NRF: U1.8 (IRQ)
- no-connect marks 13 -> 6
Other:
- note added: "Buttons"
- note added: "Comms breakout"
- note added: "SPI oled\nvertical SD cards\nBetter GPS mgnt\nBetter cabling\nMore temp sense\nPull out SPI + I2c port for future\nmcu voltage watchdog\nBarometer\nfuktighet?\n"
- note added: "Wireless"
- note removed: "Needs seperate LDO"
- note removed: "PH sensor"
- note removed: "SPI oled\nvertical SD cards\nBetter GPS mgnt\nBetter cabling\nMore temp sense\nPull out SPI + I2c port for future\nmcu voltage watchdog\n"
- note removed: "addr:0x18"
- note removed: "instead of Backup bat"
- moved on the sheet: C16, C19, C20, C21, J4, M1, R10, R9, U10A, U10B, U8
